File: pcb/pcb_nodo.sch (KiCad schematic (older format))
At the start: 24 parts, among them J1 Conn_01x02, J2 Conn_01x02, J3 Conn_01x03, J4 Conn_01x04, J5 Conn_01x18, J6 Conn_01x18, J7 UART_0, K1 FINDER-36.11, Q1 2N2219, Q2 2N2219, SW1 SW_Push, SW2 SW_Push, U1 DHT11

Commit message: 2
Parts:
- added F1: Fuse, Fuse:Fuse_Littelfuse-LVR100, symbol Device:Fuse
- added RV1: Varistor, Varistor:RV_Disc_D15.5mm_W3.9mm_P7.5mm, symbol Device:Varistor
- D1: footprint (none) -> Diode_THT:D_DO-41_SOD81_P7.62mm_Horizontal
- D2, D4: footprint (none) -> LED_THT:LED_D5.0mm_IRGrey
- D3, D5: footprint (none) -> LED_THT:LED_D3.0mm_FlatTop
- J1, J2, SW1: footprint (none) -> TerminalBlock:TerminalBlock_bornier-2_P5.08mm
- J3: footprint (none) -> Connector_PinSocket_2.54mm:PinSocket_1x03_P2.54mm_Vertical
- J4: footprint (none) -> Connector_PinSocket_2.54mm:PinSocket_1x04_P2.54mm_Vertical
- J5, J6: footprint (none) -> Connector_PinSocket_2.54mm:PinSocket_1x18_P2.54mm_Vertical
- J7: footprint (none) -> Connector_PinSocket_2.54mm:PinSocket_1x02_P2.54mm_Vertical
- Q1, Q2: footprint Package_TO_SOT_THT:TO-39-3 -> Package_TO_SOT_THT:TO-92_Inline
- R1, R2, R4, R5: footprint (none) -> Resistor_THT:R_Axial_DIN0309_L9.0mm_D3.2mm_P12.70mm_Horizontal
- R3: value R -> 10; footprint (none) -> Resistor_THT:R_Axial_DIN0309_L9.0mm_D3.2mm_P12.70mm_Horizontal
- SW2: footprint (none) -> Connector_PinHeader_2.54mm:PinHeader_1x02_P2.54mm_Vertical
Connections:
- net 13: now also SW2.1; no longer SW2.2
- net 33: now also SW1.1; no longer SW1.2
- net GND: now also SW1.2, SW2.2; no longer SW1.1, SW2.1
- net at PS1.1 (AC/L): now also F1.1, RV1.1; no longer J1.1 (Pin_1)
- net at J1.2 (Pin_2), PS1.2 (AC/N): now also RV1.2
- new net: F1.2, J1.1 (Pin_1)
Other:
- note added: "Info de temperatura"
- note added: "Pines analógicos.\nSolo entradas"
- moved on the sheet: D3, D5, J1, R4, R5, SW1, U1

Commit message: enrutado
Parts:
- F1: footprint Fuse:Fuse_Littelfuse-LVR100 -> Fuse:Fuseholder_Cylinder-5x20mm_Schurter_0031_8201_Horizontal_Open
- RV1: footprint Varistor:RV_Disc_D15.5mm_W3.9mm_P7.5mm -> Varistor:RV_Disc_D7mm_W3.4mm_P5mm
Changed lines of the file:
@@
 Wire Wire Line
 	2650 1450 2800 1450
-Text Notes 1350 900  0    118  ~ 0
+Text Notes 1350 850  0    118  ~ 0
 Conversor AC/DC
 Wire Wire Line
@@
 F 0 "F1" V 1253 1250 50  0000 C CNN
 F 1 "Fuse" V 1344 1250 50  0000 C CNN
-F 2 "Fuse:Fuse_Littelfuse-LVR100" V 1380 1250 50  0001 C CNN
+F 2 "Fuse:Fuseholder_Cylinder-5x20mm_Schurter_0031_8201_Horizontal_Open" V 1380 1250 50  0001 C CNN
 F 3 "~" H 1450 1250 50  0001 C CNN
 	1    1450 1250
@@
 F 0 "RV1" H 1400 1300 50  0000 L CNN
 F 1 "Varistor" H 1350 1400 50  0000 L CNN
-F 2 "Varistor:RV_Disc_D15.5mm_W3.9mm_P7.5mm" V 1630 1550 50  0001 C CNN
+F 2 "Varistor:RV_Disc_D7mm_W3.4mm_P5mm" V 1630 1550 50  0001 C CNN
 F 3 "~" H 1700 1550 50  0001 C CNN
 	1    1700 1550

Commit message: avances
Parts:
- Q1, Q2: footprint Package_TO_SOT_THT:TO-92_Inline -> Package_TO_SOT_THT:TO-92_Inline_Wide
Connections:
- net 12 renamed led1
- net 13 renamed pulsador2
- net 17 renamed salidarelay
- net 2 renamed salidair
- net 23 renamed temp
- net 25 renamed led2
- net 33 renamed pulsador1
Other:
- note added: "100 mA"
- note added: "220v"
- moved on the sheet: J3
Changed lines of the file:
@@
 Sheet 1 1
 Title "Smart Public Buildings - Node"
-Date "2020-09-24"
+Date "2020-10-14"
 Rev "1.0"
 Comp "Lucas Monzón Languasco - SuSTI"
 Comment1 "Shield Heltec LoRa "
-Comment2 ""
-Comment3 ""
-Comment4 ""
+Comment2 "Revisor alumno : Daniel Marquez"
+Comment3 "Revisor docente : Diego Brengi"
+Comment4 "Licencia BSD (proyecto CIAA), GPL o OHL (Cern)."
 $EndDescr
 $Comp
@@
 NoConn ~ 6700 2500
 Text Label 6900 2200 0    50   ~ 0
-23
+temp
 Wire Wire Line
 	6900 2200 6700 2200
@@
 NoConn ~ 6700 1900
 Text Label 6900 1800 0    50   ~ 0
-2
+salidair
 NoConn ~ 6700 1700
 Text Label 6900 1600 0    50   ~ 0
-17
+salidarelay
 NoConn ~ 6700 1500
 Wire Wire Line
@@
 NoConn ~ 5550 2500
 NoConn ~ 5550 2400
-Text Label 5250 2300 0    50   ~ 0
+Text Label 4750 2300 0    50   ~ 0
 32
-Text Label 5250 2200 0    50   ~ 0
-33
-Text Label 5250 2100 0    50   ~ 0
-25
+Text Label 4750 2200 0    50   ~ 0
+pulsador1
 NoConn ~ 5550 2000
 NoConn ~ 5550 1900
 NoConn ~ 5550 1800
-Text Label 5250 1700 0    50   ~ 0
-12
+Text Label 5100 1700 0    50   ~ 0
+led1
 NoConn ~ 5550 1500
-Text Label 5250 1600 0    50   ~ 0
-13
-Wire Wire Line
-	5250 1600 5550 1600
-Wire Wire Line
-	5250 1700 5550 1700
-Wire Wire Line
-	5250 2100 5550 2100
-Wire Wire Line
-	5250 2200 5550 2200
-Wire Wire Line
-	5250 2300 5550 2300
+Text Label 5100 1600 0    50   ~ 0
+pulsador2
 Wire Wire Line
 	5250 2600 5550 2600
@@
 	1    0    0    -1
 $EndComp
-Text Label 2750 3300 1    79   ~ 0
-23
 Wire Wire Line
 	2500 3300 2750 3300
@@
 	6900 5800 7350 5800
 Text Label 6150 5800 2    79   ~ 0
-13
+pulsador2
 Wire Wire Line
 	6500 5800 6150 5800
@@
 $EndComp
 $Comp
-L Relay:FINDER-36.11 K1
-U 1 1 5F702DB2
-P 2900 5600
-F 0 "K1" H 2900 5050 50  0000 L CNN
-F 1 "FINDER-36.11" H 2650 4950 50  0000 L CNN
-F 2 "Relay_THT:Relay_SPDT_Finder_36.11" H 4170 5570 50  0001 C CNN
-F 3 "https://gfinder.findernet.com/public/attachments/36/EN/S36EN.pdf" H 2900 5600 50  0001 C CNN
-	1    2900 5600
-	1    0    0    -1
-$EndComp
-$Comp
 L Transistor_BJT:2N2219 Q1
 U 1 1 5F726CB5
@@
 F 0 "Q1" H 2140 6546 50  0000 L CNN
 F 1 "2N2219" H 2140 6455 50  0000 L CNN
-F 2 "Package_TO_SOT_THT:TO-92_Inline" H 2150 6425 50  0001 L CIN
+F 2 "Package_TO_SOT_THT:TO-92_Inline_Wide" H 2150 6425 50  0001 L CIN
 F 3 "http://www.onsemi.com/pub_link/Collateral/2N2219-D.PDF" H 1950 6500 50  0001 L CNN
 	1    1950 6500
 	1    0    0    -1
 $EndComp
-Text Label 1150 6500 2    79   ~ 0
-17
+Text Label 1150 6500 1    79   ~ 0
+salidarelay
 $Comp
 L Device:D D1
@@
 	2050 5100 2050 5400
 Wire Wire Line
-	2700 5850 2700 5900
-Wire Wire Line
 	2700 6050 2050 6050
 Wire Wire Line
@@
 	1350 6500 1150 6500
 Wire Wire Line
-	3100 6050 3100 5900
-Wire Wire Line
 	3600 5600 3600 6050
 Wire Wire Line
-	3600 6050 3100 6050
-Wire Wire Line
 	3600 5500 3600 5100
 Wire Wire Line
 	3600 5100 3200 5100
-Connection ~ 3100 5900
-Wire Wire Line
-	3100 5900 3100 5850
-Connection ~ 2700 5900
-Wire Wire Line
-	2700 5900 2700 6050
 Wire Wire Line
 	2700 5100 2700 5300
@@
 F 0 "Q2" H 9940 2846 50  0000 L CNN
 F 1 "2N2219" H 9940 2755 50  0000 L CNN
-F 2 "Package_TO_SOT_THT:TO-92_Inline" H 9950 2725 50  0001 L CIN
+F 2 "Package_TO_SOT_THT:TO-92_Inline_Wide" H 9950 2725 50  0001 L CIN
 F 3 "http://www.onsemi.com/pub_link/Collateral/2N2219-D.PDF" H 9750 2800 50  0001 L CNN
 	1    9750 2800
@@
 Wire Wire Line
 	9850 3000 9850 3350
-Text Label 8850 2800 0    79   ~ 0
-2
+Text Label 8850 2800 1    79   ~ 0
+salidair
 Wire Wire Line
 	9100 2800 8850 2800
@@
 Wire Wire Line
 	8950 4600 9300 4600
-Text Label 8950 4600 1    79   ~ 0
-12
 Wire Wire Line
 	9600 4600 9850 4600
@@
 U 1 1 5F7061FF
 P 5050 2800
-F 0 "J4" H 5350 2600 50  0000 C CNN
-F 1 "Conn_01x04" H 5350 2700 50  0000 C CNN
+F 0 "J4" H 5200 2400 50  0000 C CNN
+F 1 "Conn_01x04" H 5200 2500 50  0000 C CNN
 F 2 "Connector_PinSocket_2.54mm:PinSocket_1x04_P2.54mm_Vertical" H 5050 2800 50  0001 C CNN
 F 3 "~" H 5050 2800 50  0001 C CNN
@@
 L Connector_Generic:Conn_01x03 J3
 U 1 1 5F71EDAB
-P 5050 2200
-F 0 "J3" H 5350 2100 50  0000 C CNN
-F 1 "Conn_01x03" H 5350 2200 50  0000 C CNN
-F 2 "Connector_PinSocket_2.54mm:PinSocket_1x03_P2.54mm_Vertical" H 5050 2200 50  0001 C CNN
-F 3 "~" H 5050 2200 50  0001 C CNN
-	1    5050 2200
+P 4550 2200
+F 0 "J3" H 4550 1850 50  0000 C CNN
+F 1 "Conn_01x03" H 4550 1950 50  0000 C CNN
+F 2 "Connector_PinSocket_2.54mm:PinSocket_1x03_P2.54mm_Vertical" H 4550 2200 50  0001 C CNN
+F 3 "~" H 4550 2200 50  0001 C CNN
+	1    4550 2200
 	-1   0    0    1
 $EndComp
@@
 Wire Wire Line
 	6500 5000 6150 5000
-Text Label 6150 5000 2    79   ~ 0
-33
 Wire Wire Line
 	6900 5000 7350 5000
@@
 Wire Wire Line
 	10150 5550 10500 5550
-Text Label 8950 5550 1    79   ~ 0
-25
 Wire Wire Line
 	8950 5550 9300 5550
@@
 Wire Wire Line
 	1700 1900 1650 1900
-Wire Notes Line
-	5050 2000 5000 1800
-Wire Notes Line
-	5000 1800 4900 1800
-Text Notes 4400 1750 0    50   ~ 0
+Text Notes 4250 2750 0    50   ~ 0
 Pines analógicos.\nSolo entradas
-Wire Notes Line
-	5050 2500 5050 2400
 Text Notes 1150 2700 0    118  ~ 0
 Sensor de temperatura
@@
 Text Notes 2650 3600 0    50   ~ 0
 Info de temperatura
+Wire Wire Line
+	2700 5900 2700 6050
+Wire Wire Line
+	3600 6050 3100 6050
+$Comp
+L Relay:FINDER-36.11 K1
+U 1 1 5F702DB2
+P 2900 5600
+F 0 "K1" H 2900 5050 50  0000 L CNN
+F 1 "FINDER-36.11" H 2650 4950 50  0000 L CNN
+F 2 "Relay_THT:Relay_SPDT_Finder_36.11" H 4170 5570 50  0001 C CNN
+F 3 "https://gfinder.findernet.com/public/attachments/36/EN/S36EN.pdf" H 2900 5600 50  0001 C CNN
+	1    2900 5600
+	1    0    0    -1
+$EndComp
+Wire Wire Line
+	3100 5900 3100 6050
+Text Notes 950  1850 0    50   ~ 0
+220v
+Text Notes 900  1950 0    50   ~ 0
+100 mA
+Wire Notes Line
+	1050 1700 1050 1750
+Text Label 6150 5000 2    79   ~ 0
+pulsador1
+Wire Wire Line
+	4750 2200 5550 2200
+Text Label 4750 2100 0    50   ~ 0
+led2
+Wire Wire Line
+	5100 1600 5550 1600
+Wire Wire Line
+	4750 2100 5550 2100
+Wire Wire Line
+	4750 2300 5550 2300
+Text Label 8950 4600 1    79   ~ 0
+led1
+Wire Wire Line
+	5100 1700 5550 1700
+Text Label 8950 5550 1    79   ~ 0
+led2
+Wire Notes Line
+	4800 2750 4950 2750
+Text Label 2750 3300 0    79   ~ 0
+temp
 $EndSCHEMATC

Commit message: para revision
Parts:
- added H1, H2: MountingHole, MountingHole:MountingHole_2.5mm_Pad, symbol Mechanical:MountingHole
Other:
- note added: "Circuito Led IR para encendido\ny apagado de aire acondicionado"
- note added: "Circuito de relay manejado por el pulsador 1"
- note added: "Elementos mecanicos"
- note added: "Leds de estados de conexion\ny funcionamiento"
- note added: "No es necesario conectar\ndebido a que se usa siempre el\ncontacto normal abierto"
- note added: "Pines de conexion a la pcb externa (heltec lora v2)"
- note added: "Pulsadores para:\n1) encendido y apagado de luz\n2) cambios de modo y conexion a la central"
- note removed: "Circuito led IR"
- note removed: "Circuito relay"
- note removed: "Conectores"
- note removed: "Led estado de conexion"
- note removed: "Pulsadores"
- moved on the sheet: D3, D5, R4, R5, SW1
Changed lines of the file:
@@
 Wire Wire Line
 	5250 2900 5550 2900
-Text Notes 5650 950  0    118  ~ 0
-Conectores
+Text Notes 4500 950  0    79   ~ 0
+Pines de conexion a la pcb externa (heltec lora v2)
 $Comp
 L power:+3.3V #PWR0108
@@
 L power:GND #PWR0110
 U 1 1 5F6D800D
-P 10500 4850
-F 0 "#PWR0110" H 10500 4600 50  0001 C CNN
-F 1 "GND" H 10505 4677 50  0000 C CNN
-F 2 "" H 10500 4850 50  0001 C CNN
-F 3 "" H 10500 4850 50  0001 C CNN
-	1    10500 4850
+P 10500 4950
+F 0 "#PWR0110" H 10500 4700 50  0001 C CNN
+F 1 "GND" H 10505 4777 50  0000 C CNN
+F 2 "" H 10500 4950 50  0001 C CNN
+F 3 "" H 10500 4950 50  0001 C CNN
+	1    10500 4950
 	1    0    0    -1
 $EndComp
@@
 Wire Wire Line
 	3200 5100 3200 5300
-Text Notes 2200 4450 0    118  ~ 0
-Circuito relay
+Text Notes 1400 4450 0    79   ~ 0
+Circuito de relay manejado por el pulsador 1
 $Comp
 L Device:R R3
@@
 	9100 2800 8850 2800
 Wire Wire Line
-	10150 4600 10500 4600
-Text Notes 8700 4150 0    118  ~ 0
-Led estado de conexion
-Wire Wire Line
-	8950 4600 9300 4600
-Wire Wire Line
-	9600 4600 9850 4600
+	10150 4700 10500 4700
+Text Notes 8900 4200 0    79   ~ 0
+Leds de estados de conexion\ny funcionamiento
+Wire Wire Line
+	8950 4700 9300 4700
+Wire Wire Line
+	9600 4700 9850 4700
 $Comp
 L Device:R R4
 U 1 1 5F6CF01A
-P 9450 4600
-F 0 "R4" V 9650 4550 50  0000 L CNN
-F 1 "220" V 9550 4500 50  0000 L CNN
-F 2 "Resistor_THT:R_Axial_DIN0309_L9.0mm_D3.2mm_P12.70mm_Horizontal" V 9380 4600 50  0001 C CNN
-F 3 "~" H 9450 4600 50  0001 C CNN
-	1    9450 4600
+P 9450 4700
+F 0 "R4" V 9650 4650 50  0000 L CNN
+F 1 "220" V 9550 4600 50  0000 L CNN
+F 2 "Resistor_THT:R_Axial_DIN0309_L9.0mm_D3.2mm_P12.70mm_Horizontal" V 9380 4700 50  0001 C CNN
+F 3 "~" H 9450 4700 50  0001 C CNN
+	1    9450 4700
 	0    -1   -1   0
 $EndComp
@@
 L Device:LED D3
 U 1 1 5F6CA9E7
-P 10000 4600
-F 0 "D3" H 10050 4500 50  0000 R CNN
-F 1 "LED" H 10050 4400 50  0000 R CNN
-F 2 "LED_THT:LED_D3.0mm_FlatTop" H 10000 4600 50  0001 C CNN
-F 3 "~" H 10000 4600 50  0001 C CNN
-	1    10000 4600
+P 10000 4700
+F 0 "D3" H 10050 4600 50  0000 R CNN
+F 1 "LED" H 10050 4500 50  0000 R CNN
+F 2 "LED_THT:LED_D3.0mm_FlatTop" H 10000 4700 50  0001 C CNN
+F 3 "~" H 10000 4700 50  0001 C CNN
+	1    10000 4700
 	-1   0    0    1
 $EndComp
@@
 Wire Wire Line
 	3600 5600 3850 5600
-Text Notes 6250 4450 0    118  ~ 0
-Pulsadores
-Wire Wire Line
-	6500 5000 6150 5000
-Wire Wire Line
-	6900 5000 7350 5000
+Text Notes 5350 4650 0    79   ~ 0
+Pulsadores para:\n1) encendido y apagado de luz\n2) cambios de modo y conexion a la central
+Wire Wire Line
+	6500 5100 6150 5100
+Wire Wire Line
+	6900 5100 7350 5100
 $Comp
 L power:GND #PWR0115
 U 1 1 5F6AF809
-P 7350 5150
-F 0 "#PWR0115" H 7350 4900 50  0001 C CNN
-F 1 "GND" H 7355 4977 50  0000 C CNN
-F 2 "" H 7350 5150 50  0001 C CNN
-F 3 "" H 7350 5150 50  0001 C CNN
-	1    7350 5150
+P 7350 5250
+F 0 "#PWR0115" H 7350 5000 50  0001 C CNN
+F 1 "GND" H 7355 5077 50  0000 C CNN
+F 2 "" H 7350 5250 50  0001 C CNN
+F 3 "" H 7350 5250 50  0001 C CNN
+	1    7350 5250
 	1    0    0    -1
 $EndComp
@@
 L Switch:SW_Push SW1
 U 1 1 5F6ACD07
-P 6700 5000
-F 0 "SW1" H 6700 5285 50  0000 C CNN
-F 1 "SW_Push" H 6700 5194 50  0000 C CNN
-F 2 "TerminalBlock:TerminalBlock_bornier-2_P5.08mm" H 6700 5200 50  0001 C CNN
-F 3 "~" H 6700 5200 50  0001 C CNN
-	1    6700 5000
+P 6700 5100
+F 0 "SW1" H 6700 5385 50  0000 C CNN
+F 1 "SW_Push" H 6700 5294 50  0000 C CNN
+F 2 "TerminalBlock:TerminalBlock_bornier-2_P5.08mm" H 6700 5300 50  0001 C CNN
+F 3 "~" H 6700 5300 50  0001 C CNN
+	1    6700 5100
 	1    0    0    -1
 $EndComp
@@
 Wire Notes Line
 	8700 650  10850 650
-Text Notes 9150 1000 0    118  ~ 0
-Circuito led IR
+Text Notes 8800 1000 0    79   ~ 0
+Circuito Led IR para encendido\ny apagado de aire acondicionado
 Wire Wire Line
 	9850 1350 9850 1550
@@
 L Device:R R5
 U 1 1 5F9B0408
-P 9450 5550
-F 0 "R5" V 9650 5500 50  0000 L CNN
-F 1 "220" V 9550 5450 50  0000 L CNN
-F 2 "Resistor_THT:R_Axial_DIN0309_L9.0mm_D3.2mm_P12.70mm_Horizontal" V 9380 5550 50  0001 C CNN
-F 3 "~" H 9450 5550 50  0001 C CNN
-	1    9450 5550
+P 9450 5450
+F 0 "R5" V 9650 5400 50  0000 L CNN
+F 1 "220" V 9550 5350 50  0000 L CNN
+F 2 "Resistor_THT:R_Axial_DIN0309_L9.0mm_D3.2mm_P12.70mm_Horizontal" V 9380 5450 50  0001 C CNN
+F 3 "~" H 9450 5450 50  0001 C CNN
+	1    9450 5450
 	0    -1   -1   0
 $EndComp
@@
 L Device:LED D5
 U 1 1 5F9B0796
-P 10000 5550
-F 0 "D5" H 10039 5432 50  0000 R CNN
-F 1 "LED" H 10050 5350 50  0000 R CNN
-F 2 "LED_THT:LED_D3.0mm_FlatTop" H 10000 5550 50  0001 C CNN
-F 3 "~" H 10000 5550 50  0001 C CNN
-	1    10000 5550
+P 10000 5450
+F 0 "D5" H 10039 5332 50  0000 R CNN
+F 1 "LED" H 10050 5250 50  0000 R CNN
+F 2 "LED_THT:LED_D3.0mm_FlatTop" H 10000 5450 50  0001 C CNN
+F 3 "~" H 10000 5450 50  0001 C CNN
+	1    10000 5450
 	-1   0    0    1
 $EndComp
@@
 L power:GND #PWR03
 U 1 1 5F9B0D61
-P 10500 5750
-F 0 "#PWR03" H 10500 5500 50  0001 C CNN
-F 1 "GND" H 10505 5577 50  0000 C CNN
-F 2 "" H 10500 5750 50  0001 C CNN
-F 3 "" H 10500 5750 50  0001 C CNN
-	1    10500 5750
-	1    0    0    -1
-$EndComp
-Wire Wire Line
-	9600 5550 9850 5550
-Wire Wire Line
-	10150 5550 10500 5550
-Wire Wire Line
-	8950 5550 9300 5550
+P 10500 5650
+F 0 "#PWR03" H 10500 5400 50  0001 C CNN
+F 1 "GND" H 10505 5477 50  0000 C CNN
+F 2 "" H 10500 5650 50  0001 C CNN
+F 3 "" H 10500 5650 50  0001 C CNN
+	1    10500 5650
+	1    0    0    -1
+$EndComp
+Wire Wire Line
+	9600 5450 9850 5450
+Wire Wire Line
+	10150 5450 10500 5450
+Wire Wire Line
+	8950 5450 9300 5450
 $Comp
 L Device:Fuse F1
@@
 	1650 1900 1650 1950
 Wire Wire Line
-	10500 4600 10500 4850
-Wire Wire Line
-	10500 5550 10500 5750
-Wire Wire Line
-	7350 5000 7350 5150
+	10500 4700 10500 4950
+Wire Wire Line
+	10500 5450 10500 5650
+Wire Wire Line
+	7350 5100 7350 5250
 Wire Wire Line
 	7350 5800 7350 5950
@@
 Wire Notes Line
 	1050 1700 1050 1750
-Text Label 6150 5000 2    79   ~ 0
+Text Label 6150 5100 2    79   ~ 0
 pulsador1
 Wire Wire Line
@@
 Wire Wire Line
 	4750 2300 5550 2300
-Text Label 8950 4600 1    79   ~ 0
+Text Label 8950 4700 1    79   ~ 0
 led1
 Wire Wire Line
 	5100 1700 5550 1700
-Text Label 8950 5550 1    79   ~ 0
+Text Label 8950 5450 1    79   ~ 0
 led2
 Wire Notes Line
@@
 Text Label 2750 3300 0    79   ~ 0
 temp
+$Comp
+L Mechanical:MountingHole H1
+U 1 1 5F88EA7D
+P 5350 6850
+F 0 "H1" H 5450 6896 50  0000 L CNN
+F 1 "MountingHole" H 5450 6805 50  0000 L CNN
+F 2 "MountingHole:MountingHole_2.5mm_Pad" H 5350 6850 50  0001 C CNN
+F 3 "~" H 5350 6850 50  0001 C CNN
+	1    5350 6850
+	1    0    0    -1
+$EndComp
+$Comp
+L Mechanical:MountingHole H2
+U 1 1 5F88ED2A
+P 6200 6850
+F 0 "H2" H 6300 6896 50  0000 L CNN
+F 1 "MountingHole" H 6300 6805 50  0000 L CNN
+F 2 "MountingHole:MountingHole_2.5mm_Pad" H 6200 6850 50  0001 C CNN
+F 3 "~" H 6200 6850 50  0001 C CNN
+	1    6200 6850
+	1    0    0    -1
+$EndComp
+Wire Notes Line width 8 style solid
+	6900 7050 5100 7050
+Wire Notes Line width 8 style solid
+	5100 7050 5100 6450
+Wire Notes Line width 8 style solid
+	5100 6450 6900 6450
+Text Notes 5400 6600 0    79   ~ 0
+Elementos mecanicos
+Wire Notes Line width 8 style solid
+	6900 6450 6900 7050
+Wire Notes Line
+	3000 5200 3250 4850
+Text Notes 3250 4900 0    59   ~ 0
+No es necesario conectar\ndebido a que se usa siempre el\ncontacto normal abierto
 $EndSCHEMATC
